File: dock/vocore_dock.sch (EAGLE design)
At the start: 31 parts

Commit message: adding gnd's
Connections:
- net GND: now also MICROSD.GND@0, MICROSD.GND@1, RJ45.GND
Changed lines of the file:
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@@
 <pinref part="GND3" gate="1" pin="GND"/>
 <wire x1="-63.5" y1="15.24" x2="-63.5" y2="12.7" width="0.1524" layer="91"/>
+<pinref part="RJ45" gate="G$1" pin="GND"/>
+<wire x1="-38.1" y1="15.24" x2="-63.5" y2="15.24" width="0.1524" layer="91"/>
 </segment>
 <segment>
@@
 <wire x1="12.7" y1="-81.28" x2="7.62" y2="-81.28" width="0.1524" layer="91"/>
 <pinref part="GND6" gate="1" pin="GND"/>
+<pinref part="MICROSD" gate="G$1" pin="GND@1"/>
+<wire x1="15.24" y1="-81.28" x2="12.7" y2="-81.28" width="0.1524" layer="91"/>
+<pinref part="MICROSD" gate="G$1" pin="GND@0"/>
+<wire x1="15.24" y1="-83.82" x2="12.7" y2="-83.82" width="0.1524" layer="91"/>
 </segment>
 <segment>
